File: Hardware/InkTime.brd (EAGLE design)
At the start: 46 x 35.1 mm, 105 parts, among them IC1 BQ25180YBGR_BQ25180YBGRBQ2518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, IC2 DRV2605YZFR_DRV2605YZFR, IC3 BMA423_BMA423, IC9 RT6160AWSC_RT6160AWSC, J1 503480-2400_503480-2400, J2 TC2030-IDC_TC2030-IDC, J3 KH-TYPE-C-16P_KH-TYPE-C-16P, Q1 20V/4.2A/52mΩ/1.4W, Q3 ESP32_C6_LIBRARY_6_SI1308EDL-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, U1 NORDIC_NRF_4_NRF52840_QF, U3 ESP32_C6_LIBRARY_MAX17048G+T10, X1 32MHz, X2 32.768kHz

Commit message: Am rezolvat issue-urile din review
Parts:
- moved ANT1 3.75 mm to (19.6, 11.7)
Routing:
- net RF: track 20.6 -> 16.9 mm
- net SWDCLK: track 27.5 -> 25.4 mm
Other:
- outline, holes or cut-outs redrawn
